Commit message: added some simulation files

File: description/gazebo_control.xacro (robot description, xacro)
@@ -5,7 +5,5 @@
             <!-- Wheel Information -->
             <left_joint>left_wheel_joint</left_joint>
-            <left_joint>left_back_joint</left_joint>
             <right_joint>right_wheel_joint</right_joint>
-            <right_joint>right_wheel_back_joint</right_joint>
             <wheel_separation>0.297</wheel_separation>
             <wheel_diameter>0.066</wheel_diameter>

File: description/lidar.xacro (robot description, xacro)
@@ -23,3 +23,31 @@
         </xacro:inertial_cylinder>
     </link>
+    <gazebo reference="lidar_frame">
+        <material>Gazebo/Black</material>
+        <sensor name="laser" type="ray">
+            <pose> 0 0 0 0 0 0 </pose>
+            <visualize>false</visualize>
+            <update_rate>10</update_rate>
+            <ray>
+                <scan>
+                    <horizontal>
+                        <samples>360</samples>
+                        <min_angle>-3.14</min_angle>
+                        <max_angle>3.14</max_angle>
+                    </horizontal>
+                </scan>
+                <range>
+                    <min>0.3</min>
+                    <max>12</max>
+                </range>
+            </ray>
+            <plugin name="laser_controller" filename="libgazebo_ros_ray_sensor.so">
+                <ros>
+                    <argument>~/out:=scan</argument>
+                </ros>
+                <output_type>sensor_msgs/LaserScan</output_type>
+                <frame_name>laser_frame</frame_name>
+            </plugin>
+        </sensor>
+    </gazebo>
 </robot>

File: description/robot.urdf.xacro (robot description, xacro)
@@ -1,6 +1,13 @@
 <?xml version="1.0"?>
 <robot xmlns:xacro="http://www.ros.org/wiki/xacro"  name="robot">
+    <xacro:arg name="use_ros2_control" default="true"/>
+    <xacro:arg name="sim_mode" default="true"/>
     <xacro:include filename="robot_core.xacro" />
+    <xacro:if value="$(arg use_ros2_control)">
+        <xacro:include filename="ros2_control.xacro" />
+    </xacro:if>
+    <xacro:unless value="$(arg use_ros2_control)">
+        <xacro:include filename="gazebo_control.xacro" />
+    </xacro:unless>
     <xacro:include filename="lidar.xacro" />
-    <xacro:include filename="ros2_control.xacro"/>
 </robot>

File: description/robot_core.xacro (robot description, xacro)
@@ -3,5 +3,5 @@
     <xacro:include filename="inertial_macros.xacro"/>
     <material name="white">
-        <color rgba="1 1 1 1"/>
+        <color rgba="1 1 1 1" />
     </material>
     <material name="orange">
@@ -13,4 +13,7 @@
     <material name="black">
         <color rgba="0 0 0 1"/>
+    </material>
+    <material name="red">
+        <color rgba="1 0 0 1"/>
     </material>
     <!-- BASE LINK -->
@@ -48,4 +51,7 @@
         </xacro:inertial_box>
     </link>
+    <gazebo reference="chassis">
+        <material>Gazebo/Orange</material>
+    </gazebo>
     <!-- LEFT WHEEL FRONT LINK -->
     <joint name="left_wheel_joint" type="continuous">
@@ -74,4 +80,7 @@
         </xacro:inertial_cylinder>
     </link>
+    <gazebo reference="left_wheel">
+        <material>Gazebo/Blue</material>
+    </gazebo>
     <!-- LEFT WHEEL BACK LINK -->
     <!--
@@ -128,4 +137,7 @@
         </xacro:inertial_cylinder>
     </link>
+    <gazebo reference="right_wheel">
+        <material>Gazebo/Blue</material>
+    </gazebo>
      <!-- RIGHT WHEEL BACK LINK -->
      <!--

File: description/ros2_control.xacro (robot description, xacro)
@@ -1,85 +1,72 @@
 <?xml version="1.0"?>
 <robot xmlns:xacro="http://www.ros.org/wiki/xacro">
-    <ros2_control name="RealRobot" type="system">
-        <hardware>
-            <plugin>roboclaw_hardware_interface/RoboClawHardwareInterface</plugin>
-            <param name="serial_port">/dev/ttyACM0</param>
-            <param name="serial_baud" type="int">38400</param>
-          </hardware>
-        <joint name="left_wheel_joint">
-            <command_interface name="velocity"/>
-            <state_interface name="position"/>
-            <param name="address">128</param>
-            <param name="qppr">500</param>
-            <param name="motor_type">M2</param>
-        </joint>
-        <!--
-        <joint name="left_back_joint">
-            <command_interface name="velocity"/>
-            <state_interface name="position"/>
-            <param name="address">128</param>
-            <param name="qppr">500</param>
-            <param name="motor_type">M2</param>
-        </joint>
-        -->
-        <joint name="right_wheel_joint">
-            <command_interface name="velocity"/>
-            <state_interface name="position"/>
-            <param name="address">128</param>
-            <param name="qppr">500</param>
-            <param name="motor_type">M1</param>
-        </joint>
-        <!--
-        <joint name="right_wheel_back_joint">
-            <command_interface name="velocity"/>
-            <state_interface name="position"/>
-            <param name="address">128</param>
-            <param name="qppr">500</param>
-            <param name="motor_type">M1</param>
-        </joint>
-        -->
-    </ros2_control>
-    <!--
-    <ros2_control name="GazeboSystem" type="system">
-        <hardware>
-            <plugin>gazebo_ros2_control/GazeboSystem</plugin>
-        </hardware>
-        <joint name="left_wheel_joint">
-            <command_interface name="velocity">
-                <param name ="min">-10</param>
-                <param name ="max">10</param>
-            </command_interface>
-            <state_interface name="velocity"/>
-            <state_interface name="position"/>
-        </joint>
-        <joint name="left_back_joint">
-            <command_interface name="velocity">
-                <param name ="min">-10</param>
-                <param name ="max">10</param>
-            </command_interface>
-            <state_interface name="velocity"/>
-            <state_interface name="position"/>
-        </joint>
-        <joint name="right_wheel_joint">
-            <command_interface name="velocity">
-                <param name ="min">-10</param>
-                <param name ="max">10</param>
-            </command_interface>
-            <state_interface name="velocity"/>
-            <state_interface name="position"/>
-        </joint>
-        <joint name="right_wheel_back_joint">
-            <command_interface name="velocity">
-                <param name ="min">-10</param>
-                <param name ="max">10</param>
-            </command_interface>
-            <state_interface name="velocity"/>
-            <state_interface name="position"/>
-        </joint>
-    </ros2_control>
-    -->
+    <xacro:unless value="$(arg sim_mode)">
+        <ros2_control name="RealRobot" type="system">
+            <hardware>
+                <plugin>roboclaw_hardware_interface/RoboClawHardwareInterface</plugin>
+                <param name="serial_port">/dev/ttyACM0</param>
+                <param name="serial_baud" type="int">38400</param>
+              </hardware>
+            <joint name="left_wheel_joint">
+                <command_interface name="velocity"/>
+                <state_interface name="position"/>
+                <param name="address">128</param>
+                <param name="qppr">500</param>
+                <param name="motor_type">M2</param>
+            </joint>
+            <!--
+            <joint name="left_back_joint">
+                <command_interface name="velocity"/>
+                <state_interface name="position"/>
+                <param name="address">128</param>
+                <param name="qppr">500</param>
+                <param name="motor_type">M2</param>
+            </joint>
+            -->
+            <joint name="right_wheel_joint">
+                <command_interface name="velocity"/>
+                <state_interface name="position"/>
+                <param name="address">128</param>
+                <param name="qppr">500</param>
+                <param name="motor_type">M1</param>
+            </joint>
+            <!--
+            <joint name="right_wheel_back_joint">
+                <command_interface name="velocity"/>
+                <state_interface name="position"/>
+                <param name="address">128</param>
+                <param name="qppr">500</param>
+                <param name="motor_type">M1</param>
+            </joint>
+            -->
+        </ros2_control>
+    </xacro:unless>
+    <xacro:if value="$(arg sim_mode)">
+        <ros2_control name="GazeboSystem" type="system">
+            <hardware>
+                <plugin>gazebo_ros2_control/GazeboSystem</plugin>
+            </hardware>
+            <joint name="left_wheel_joint">
+                <command_interface name="velocity">
+                    <param name="min">-10</param>
+                    <param name="max">10</param>
+                </command_interface>
+                <state_interface name="velocity"/>
+                <state_interface name="position"/>
+            </joint>
+            <joint name="right_wheel_joint">
+                <command_interface name="velocity">
+                    <param name="min">-10</param>
+                    <param name="max">10</param>
+                </command_interface>
+                <state_interface name="velocity"/>
+                <state_interface name="position"/>
+            </joint>
+        </ros2_control>
+    </xacro:if>
     <gazebo>
-        <plugin name="gazebo_ros2_control" filename="libgazebo_ros2_control">
+        <plugin name="gazebo_ros2_control" filename="libgazebo_ros2_control.so">
             <parameters>$(find GaiaBotRos)/config/my_controllers.yaml</parameters>
+            <parameters>$(find GaiaBotRos)/config/gaz_ros2_ctl_use_sim.yaml</parameters>
         </plugin>
     </gazebo>
