Commit message: simulation with working simulated LiDAR

File: description/lidar.xacro (robot description, xacro)
@@ -1,31 +1,37 @@
 <?xml version="1.0"?>
 <robot xmlns:xacro="http://www.ros.org/wiki/xacro" >
-    <joint name="lidar_join" type="fixed">
+    <joint name="laser_joint" type="fixed">
         <parent link="chassis"/>
-        <child link="lidar_frame"/>
-        <origin xyz="0 0 0.1" rpy="0 0 0"/>
+        <child link="laser_frame"/>
+        <origin xyz="0.122 0 0.212" rpy="0 0 0"/>
     </joint>
-    <link name="lidar_frame">
+    <link name="laser_frame">
         <visual>
-            <origin xyz="0 0 0"/>
             <geometry>
-                <cylinder radius="0.07" length="0.07"/>
+                <cylinder radius="0.05" length="0.04"/>
             </geometry>
-            <material name="orange"/>
+            <material name="red"/>
+        </visual>
+        <visual>
+            <origin xyz="0 0 -0.05"/>
+            <geometry>
+                <cylinder radius="0.01" length="0.1"/>
+            </geometry>
+            <material name="red"/>
         </visual>
         <collision>
             <geometry>
-                <cylinder radius="0.07" length="0.07"/>
+                <cylinder radius="0.05" length="0.04"/>
             </geometry>
         </collision>
-        <xacro:inertial_cylinder mass="0.25" radius="0.07" length="0.07">
+        <xacro:inertial_cylinder mass="0.1" length="0.04" radius="0.05">
             <origin xyz="0 0 0" rpy="0 0 0"/>
         </xacro:inertial_cylinder>
     </link>
-    <gazebo reference="lidar_frame">
-        <material>Gazebo/Black</material>
+    <gazebo reference="laser_frame">
+        <material>Gazebo/Red</material>
         <sensor name="laser" type="ray">
             <pose> 0 0 0 0 0 0 </pose>
-            <visualize>false</visualize>
+            <visualize>true</visualize>
             <update_rate>10</update_rate>
             <ray>

File: description/robot.urdf.xacro (robot description, xacro)
@@ -1,13 +1,6 @@
 <?xml version="1.0"?>
 <robot xmlns:xacro="http://www.ros.org/wiki/xacro"  name="robot">
-    <xacro:arg name="use_ros2_control" default="true"/>
-    <xacro:arg name="sim_mode" default="true"/>
     <xacro:include filename="robot_core.xacro" />
-    <xacro:if value="$(arg use_ros2_control)">
-        <xacro:include filename="ros2_control.xacro" />
-    </xacro:if>
-    <xacro:unless value="$(arg use_ros2_control)">
-        <xacro:include filename="gazebo_control.xacro" />
-    </xacro:unless>
     <xacro:include filename="lidar.xacro" />
+    <xacro:include filename="gazebo_control.xacro"/>
 </robot>

File: description/robot_core.xacro (robot description, xacro)
@@ -2,4 +2,18 @@
 <robot xmlns:xacro="http://www.ros.org/wiki/xacro" >
     <xacro:include filename="inertial_macros.xacro"/>
+    <xacro:property name="chassis_length" value="0.335"/>
+    <xacro:property name="chassis_width" value="0.265"/>
+    <xacro:property name="chassis_height" value="0.138"/>
+    <xacro:property name="chassis_mass" value="1.0"/>
+    <xacro:property name="wheel_radius" value="0.07"/>
+    <xacro:property name="wheel_thickness" value="0.07"/>
+    <xacro:property name="wheel_mass" value="0.2"/>
+    <xacro:property name="wheel_offset_x" value="0.33"/>
+    <xacro:property name="wheel_offset_y" value="0.1485"/>
+    <xacro:property name="wheel_offset_z" value="0.01"/>
+    <xacro:property name="caster_wheel_radius" value="0.01"/>
+    <xacro:property name="caster_wheel_mass" value="0.01"/>
+    <xacro:property name="caster_wheel_offset_x" value="0.075"/>
+    <xacro:property name="caster_wheel_offset_z" value="${wheel_offset_z - wheel_radius + caster_wheel_radius}"/>
     <material name="white">
         <color rgba="1 1 1 1" />
@@ -18,11 +32,7 @@
     </material>
     <!-- BASE LINK -->
-    <link name="base_link"></link>
-    <joint name="chassis_joint" type="fixed">
-        <parent link="base_link"/>
-        <child link="chassis"/>
-        <origin xyz="-0 0 0"/>
-    </joint>
-    <!--BASE FOOTPRINT LINK-->
+    <link name="base_link">
+    </link>
+    <!-- BASE_FOOTPRINT LINK -->
     <joint name="base_footprint_joint" type="fixed">
         <parent link="base_link"/>
@@ -33,20 +43,25 @@
     </link>
     <!-- CHASSIS LINK -->
+    <joint name="chassis_joint" type="fixed">
+        <parent link="base_link"/>
+        <child link="chassis"/>
+        <origin xyz="${-wheel_offset_x} 0 ${-wheel_offset_z}"/>
+    </joint>
     <link name="chassis">
         <visual>
-            <origin xyz="0 0 0"/>
+            <origin xyz="${chassis_length/2} 0 ${chassis_height/2}"/>
             <geometry>
-                <box size="0.23 0.27 0.15"/>
+                <box size="${chassis_length} ${chassis_width} ${chassis_height}"/>
             </geometry>
-            <material name="white"/>
+            <material name="orange"/>
         </visual>
         <collision>
-            <origin xyz="0 0 0"/>
+            <origin xyz="${chassis_length/2} 0 ${chassis_height/2}"/>
             <geometry>
-                <box size="0.23 0.27 0.15"/>
+                <box size="${chassis_length} ${chassis_width} ${chassis_height}"/>
             </geometry>
         </collision>
-        <xacro:inertial_box mass="3" x="0.23" y="0.27" z="0.15">
-            <origin xyz="0 0 0" rpy="0 0 0"/>
+        <xacro:inertial_box mass="0.5" x="${chassis_length}" y="${chassis_width}" z="${chassis_height}">
+            <origin xyz="${chassis_length/2} 0 ${chassis_height/2}" rpy="0 0 0"/>
         </xacro:inertial_box>
     </link>
@@ -54,18 +69,15 @@
         <material>Gazebo/Orange</material>
     </gazebo>
-    <!-- LEFT WHEEL FRONT LINK -->
+    <!-- LEFT WHEEL LINK -->
     <joint name="left_wheel_joint" type="continuous">
         <parent link="base_link"/>
         <child link="left_wheel"/>
-        <origin xyz="0.12 0.15 0" rpy="-${pi/2} 0 0" />
+        <origin xyz="0 ${wheel_offset_y} 0" rpy="-${pi/2} 0 0" />
         <axis xyz="0 0 1"/>
-        <command_interface name="velocity"/>
-        <state_interface name="position"/>
     </joint>
     <link name="left_wheel">
         <visual>
-            <origin xyz="0 0 0"/>
             <geometry>
-                <cylinder radius="0.07" length="0.07"/>
+                <cylinder radius="${wheel_radius}" length="${wheel_thickness}"/>
             </geometry>
             <material name="blue"/>
@@ -73,8 +85,8 @@
         <collision>
             <geometry>
-                <cylinder radius="0.07" length="0.07"/>
+                <sphere radius="${wheel_radius}"/>
             </geometry>
         </collision>
-        <xacro:inertial_cylinder mass="0.25" radius="0.07" length="0.07">
+        <xacro:inertial_cylinder mass="${wheel_mass}" length="${wheel_thickness}" radius="${wheel_radius}">
             <origin xyz="0 0 0" rpy="0 0 0"/>
         </xacro:inertial_cylinder>
@@ -83,19 +95,15 @@
         <material>Gazebo/Blue</material>
     </gazebo>
-    <!-- LEFT WHEEL BACK LINK -->
-    <!--
-    <joint name="left_back_joint" type="continuous">
+    <!-- RIGHT WHEEL LINK -->
+    <joint name="right_wheel_joint" type="continuous">
         <parent link="base_link"/>
-        <child link="left_wheel_back"/>
-        <origin xyz="-0.12 0.15 0" rpy="-${pi/2} 0 0"/>
+        <child link="right_wheel"/>
+        <origin xyz="0 ${-wheel_offset_y} 0" rpy="${pi/2} 0 0" />
         <axis xyz="0 0 -1"/>
-        <command_interface name="velocity"/>
-        <state_interface name="position"/>
     </joint>
-    <link name="left_wheel_back">
+    <link name="right_wheel">
         <visual>
-            <origin xyz="0 0 0"/>
             <geometry>
-                <cylinder radius="0.07" length="0.07"/>
+                <cylinder radius="${wheel_radius}" length="${wheel_thickness}"/>
             </geometry>
             <material name="blue"/>
@@ -103,35 +111,8 @@
         <collision>
             <geometry>
-                <cylinder radius="0.07" length="0.07"/>
+                <sphere radius="${wheel_radius}"/>
             </geometry>
         </collision>
-        <xacro:inertial_cylinder mass="0.25" radius="0.07" length="0.07">
-            <origin xyz="0 0 0" rpy="0 0 0"/>
-        </xacro:inertial_cylinder>
-    </link>
-    !-->
-    <!-- RIGHT WHEEL FRONT LINK -->
-    <joint name="right_wheel_joint" type="continuous">
-        <parent link="base_link"/>
-        <child link="right_wheel"/>
-        <origin xyz="0.12 -0.15 0" rpy="${pi/2} 0 0" />
-        <axis xyz="0 0 -1"/>
-        <command_interface name="velocity"/>
-        <state_interface name="position"/>
-    </joint>
-    <link name="right_wheel">
-        <visual>
-            <origin xyz="0 0 0"/>
-            <geometry>
-                <cylinder radius="0.07" length="0.07"/>
-            </geometry>
-            <material name="blue"/>
-        </visual>
-        <collision>
-            <geometry>
-                <cylinder radius="0.07" length="0.07"/>
-            </geometry>
-        </collision>
-        <xacro:inertial_cylinder mass="0.25" radius="0.07" length="0.07">
+        <xacro:inertial_cylinder mass="${wheel_mass}" length="${wheel_thickness}" radius="${wheel_radius}">
             <origin xyz="0 0 0" rpy="0 0 0"/>
         </xacro:inertial_cylinder>
@@ -140,19 +121,15 @@
         <material>Gazebo/Blue</material>
     </gazebo>
-     <!-- RIGHT WHEEL BACK LINK -->
-     <!--
-     <joint name="right_wheel_back_joint" type="continuous">
-        <parent link="base_link"/>
-        <child link="right_wheel_back"/>
-        <origin xyz="-0.12 -0.15 0" rpy="${pi/2} 0 0" />
+    <!-- CASTER RIGHT WHEEL LINK -->
+    <joint name="caster_right_joint" type="fixed">
+        <parent link="chassis"/>
+        <child link="caster_right"/>
+        <origin xyz="0.01 ${-wheel_offset_y} 0.01" rpy="${pi/2} 0 0" />
         <axis xyz="0 0 -1"/>
-        <command_interface name="velocity"/>
-        <state_interface name="position"/>
     </joint>
-    <link name="right_wheel_back">
+    <link name="caster_right">
         <visual>
-            <origin xyz="0 0 0"/>
             <geometry>
-                <cylinder radius="0.07" length="0.07"/>
+                <cylinder radius="${wheel_radius}" length="${wheel_thickness}"/>
             </geometry>
             <material name="blue"/>
@@ -160,11 +137,43 @@
         <collision>
             <geometry>
-                <cylinder radius="0.07" length="0.07"/>
+                <sphere radius="${wheel_radius}"/>
             </geometry>
         </collision>
-        <xacro:inertial_cylinder mass="0.25" radius="0.07" length="0.07">
+        <xacro:inertial_sphere mass="${wheel_mass}" radius="${wheel_radius}">
             <origin xyz="0 0 0" rpy="0 0 0"/>
-        </xacro:inertial_cylinder>
+        </xacro:inertial_sphere>
     </link>
-    !-->
+    <gazebo reference="caster_right">
+        <material>Gazebo/Blue</material>
+        <mu1 value="0.001"/>
+        <mu2 value="0.001"/>
+    </gazebo>
+       <!-- CASTER LEFT WHEEL LINK -->
+       <joint name="caster_left_joint" type="fixed">
+        <parent link="chassis"/>
+        <child link="caster_left"/>
+        <origin xyz="0.01 ${wheel_offset_y} 0.01" rpy="${pi/2} 0 0" />
+        <axis xyz="0 0 1"/>
+    </joint>
+    <link name="caster_left">
+        <visual>
+            <geometry>
+                <cylinder radius="${wheel_radius}" length="${wheel_thickness}"/>
+            </geometry>
+            <material name="blue"/>
+        </visual>
+        <collision>
+            <geometry>
+                <sphere radius="${wheel_radius}"/>
+            </geometry>
+        </collision>
+        <xacro:inertial_sphere mass="${wheel_mass}" radius="${wheel_radius}">
+            <origin xyz="0 0 0" rpy="0 0 0"/>
+        </xacro:inertial_sphere>
+    </link>
+    <gazebo reference="caster_left">
+        <material>Gazebo/Blue</material>
+        <mu1 value="0.001"/>
+        <mu2 value="0.001"/>
+    </gazebo>
 </robot>
